File: vintagestereo.kicad_pcb (KiCad board)
At the start: 2 copper layers, 166 x 46 mm, 8 parts

Commit message: autosync
Parts:
- removed 100s1: Mute, AA-ROB-FULL:PB86-A-Front
- removed 100s1: V12 SoundTrack, AA-ROB-FULL:PB86-A-Front
- removed 100s1: AUX, AA-ROB-FULL:PB86-A-Front
- removed 100s1: BLUTOOTH, AA-ROB-FULL:PB86-A-Front
- removed H1 (x3): MountingHole_Pad, MountingHole:MountingHole_3.2mm_M3_DIN965_Pad
- removed RADIO: PB-86A, AA-ROB-FULL:PB86-A-Front
- added J1: Conn_01x07_Male, Connector_PinHeader_2.54mm:PinHeader_1x07_P2.54mm_Vertical, F.Cu at (206.1, 70.9)
- added U1: BLUTOOTHMODULE, AA-ROB-FULL:BlutoothModule, F.Cu at (173.7, 74.8)
Routing:
- removed copper zone on F.Cu, net (none)
Other:
- board outline removed
- board text removed: "SCIMITAR"
- board text removed: "Tune"
- board text removed: "Vol"
